File: nofy_V2/nofy.kicad_pcb (KiCad board)
At the start: 2 copper layers, 214.5 x 78.9 mm, 148 parts, among them J1 PIn1x8, J10 Conn_01x01-Connector_Generic, J11 Conn_01x01-Connector_Generic, J12 Conn_01x01-Connector_Generic, J13 Conn_01x01-Connector_Generic, J14 Conn_01x01-Connector_Generic, J15 Conn_01x01-Connector_Generic, J16 Conn_01x01-Connector_Generic, J17 Conn_01x01-Connector_Generic, J18 Conn_01x01-Connector_Generic, J19 Conn_01x01-Connector_Generic, J20 Conn_01x01-Connector_Generic, J21 Conn_01x01-Connector_Generic, J22 PIn1x4, J23 PIn1x4, J24 PIn1x4, J25 PIn1x4, J26 PIn1x4, J27 PIn1x4, J28 PIn1x4, J29 PIn1x4, J30 PIn1x4, J31 PIn1x4, J32 PIn1x4, J33 PIn1x4, J34 PIn1x4, J35 PIn1x4, J36 PIn1x4, J37 PIn1x4, J38 PIn1x4, J39 PIn1x4, J40 PIn1x4, J41 PIn1x4, J7 PIn1x8, J9 PIn1x8, SW1 RotaryEncoder, SW10 SW_PUSH, SW11 SW_PUSH, SW12 SW_PUSH, SW13 SW_PUSH, SW14 SW_PUSH, SW15 SW_PUSH, SW16 SW_PUSH, SW17 SW_PUSH, SW18 SW_PUSH, SW19 SW_PUSH, SW2 RotaryEncoder, SW20 SW_PUSH, SW21 SW_PUSH, SW22 SW_PUSH, SW23 SW_PUSH, SW24 SW_PUSH, SW25 SW_PUSH, SW26 SW_PUSH, SW27 SW_PUSH, SW28 SW_PUSH, SW29 SW_PUSH, SW3 SW_SPDT, SW30 SW_PUSH, SW31 SW_PUSH, SW32 SW_PUSH, SW33 SW_PUSH, SW34 SW_PUSH, SW35 SW_PUSH, SW36 SW_PUSH, SW37 SW_PUSH, SW38 SW_PUSH, SW39 SW_PUSH, SW4 SW_SPDT, SW40 SW_PUSH, SW41 SW_PUSH, SW42 SW_PUSH, SW43 SW_PUSH, SW44 SW_PUSH, SW45 SW_PUSH, SW46 SW_PUSH, SW47 SW_PUSH, SW48 SW_PUSH, SW49 SW_PUSH, SW5 SW_PUSH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

Commit message: Add : Library
Parts:
- removed J1, J7: PIn1x8, nofy:Pin1x8
- moved J40 99.5 mm to (223.6, 149.0)
- moved J36 95.8 mm to (219.1, 148.9)
- moved J41 91.5 mm to (223.7, 159.6)
- moved J34 91.1 mm to (255.2, 150.7)
- moved J38 90.9 mm to (259.2, 149.7)
- moved J37 86.1 mm to (220.1, 160.2)
- moved J35 78.9 mm to (254.9, 162.5)
- moved J39 77.1 mm to (258.9, 163.4)
- moved SW4 18.2 mm to (276.2, 142.5)
- moved BT1 18.2 mm to (278.8, 156.8)

Commit message: Update : PCB
Parts:
- removed J9: PIn1x8, nofy:Pin1x8
- B1, BT1, SW3: moved to F.Cu
- moved J30 128.2 mm to (109.8, 46.0)
- moved J32 123.8 mm to (109.8, 61.1)
- moved J27 118.5 mm to (143.8, 54.1)
- moved J29 113.6 mm to (143.8, 69.2)
- moved J13 113.1 mm to (150.7, 28.1)
- moved J38 102.2 mm to (222.7, 54.2)
- moved J39 99.0 mm to (222.7, 71.3)
- moved J36 91.8 mm to (188.7, 62.3)
- moved J37 87.0 mm to (188.7, 79.0)
- moved D22 76.3 mm to (268.7, 143.0)
- moved D23 76.3 mm to (268.6, 160.0)
- moved SW26 76.3 mm to (267.1, 136.9)
- moved SW27 76.3 mm to (267.1, 153.9)
- moved SW28 76.3 mm to (267.1, 170.9)
- moved D24 76.3 mm to (268.8, 177.2)
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Other:
- board size 214.5 x 78.9 mm -> 249.5 x 136.4 mm

Commit message: Update : PCB
Parts:
- removed J12, J20: Conn_01x01-Connector_Generic, MountingHole:MountingHole_3.2mm_M3
- removed the REF** at (167.6, 91.5)
- added REF**: StampHole, nofy:StampHole, F.Cu at (86.3, 145.8)
- added REF**: StampHole, nofy:StampHole, F.Cu at (60.9, 141.3)
- added REF**: StampHole, nofy:StampHole, F.Cu at (119.3, 65.8)
- added REF**: StampHole, nofy:StampHole, F.Cu at (86.3, 141.3)
- added REF**: StampHole, nofy:StampHole, F.Cu at (60.9, 145.8)
- moved J17 218.9 mm to (56.6, 154.2), turned to 180 degrees
- moved J34 208.1 mm to (40.5, 182.0), turned to 180 degrees
- moved J35 203.5 mm to (40.5, 164.9), turned to 180 degrees
- moved SW4 198.8 mm to (47.6, 190.5), turned to 180 degrees
- moved SW26 184.0 mm to (84.2, 156.7), turned to -90 degrees
- moved D22 178.9 mm to (90.3, 155.1), turned to 90 degrees
- moved BT1 177.4 mm to (46.6, 162.8), turned to 0 degrees
- moved J23 172.8 mm to (101.4, 149.7), turned to 90 degrees
- moved U1 169.3 mm to (62.4, 188.1), turned to 180 degrees
- moved SW27 165.9 mm to (101.2, 156.7), turned to -90 degrees
- moved D23 161.4 mm to (107.3, 155.2), turned to 90 degrees
- moved SW28 149.6 mm to (118.2, 156.7), turned to -90 degrees
- moved D24 146.1 mm to (124.5, 155.0), turned to 90 degrees
- moved J11 141.4 mm to (92.7, 148.8), turned to 90 degrees
- moved J40 138.2 mm to (74.5, 173.9), turned to 180 degrees
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Other:
- board size 249.5 x 136.4 mm -> 205.6 x 171.6 mm
- board text added: "nofy Engine"
- board text added: "nofy V2"
- board text removed: "nofy V1"

Commit message: Update : PCB
Parts:
- renumbered REF** to REF**1, REF** to REF**2, REF** to REF**3, REF** to REF**4, REF** to REF**5
Connections:
- U3 pad 2: col5 -> Col5
- U3 pad 3: col4 -> Col4
- U3 pad 4: col3 -> Col3
- U3 pad 5: col2 -> Col2
- U3 pad 6: col1 -> Col1
- U3 pad 7: col0 -> Col0
Routing:
- net 3.3V: track 0.00 -> 171.7 mm, vias 0 -> 18
- net Row7: track 0.00 -> 169.4 mm, vias 0 -> 15
- net Row3: track 0.00 -> 150.5 mm, vias 0 -> 12
- net Row8: track 0.00 -> 149.6 mm, vias 0 -> 8
- net Col4: track 0.00 -> 139.9 mm, vias 0 -> 4
- net Row6: track 0.00 -> 138.5 mm, vias 0 -> 15
- net GND_R: track 0.00 -> 137.0 mm, vias 0 -> 9
- net Row5: track 0.00 -> 133.3 mm, vias 0 -> 9
- net Col7: track 0.00 -> 129.4 mm, vias 0 -> 5
- net Col2: track 0.00 -> 125.2 mm, vias 0 -> 6
- net Col3: track 0.00 -> 124.4 mm, vias 0 -> 8
- net SDIO: track 0.00 -> 118.0 mm, vias 0 -> 11
- net Row0: track 0.00 -> 117.7 mm, vias 0 -> 15
- net Col5: track 0.00 -> 115.3 mm, vias 0 -> 5
- net Col8: track 0.00 -> 114.8 mm, vias 0 -> 4
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