File: PCB/nofy_V2/nofy.kicad_pcb (KiCad board)
At the start: 2 copper layers, 314.7 x 88.7 mm, 166 parts, among them J18 PIn1x4, J21 PIn1x4, J32 PIn1x4, J33 PIn1x4, SW1 SW_SPDT, SW10 SW_PUSH, SW11 SW_PUSH, SW12 SW_PUSH, SW13 SW_PUSH, SW14 SW_PUSH, SW15 SW_PUSH, SW16 SW_PUSH, SW17 SW_PUSH, SW18 SW_PUSH, SW19 SW_PUSH, SW2 SW_SPDT, SW20 SW_PUSH, SW21 SW_PUSH, SW22 SW_PUSH, SW23 SW_PUSH, SW24 SW_PUSH, SW25 SW_PUSH, SW26 SW_PUSH, SW27 SW_PUSH, SW28 SW_PUSH, SW29 SW_PUSH, SW3 RotaryEncoder, SW30 SW_PUSH, SW31 SW_PUSH, SW32 SW_PUSH, SW33 SW_PUSH, SW34 SW_PUSH, SW35 SW_PUSH, SW36 SW_PUSH, SW37 SW_PUSH, SW38 SW_PUSH, SW39 SW_PUSH, SW4 RotaryEncoder, SW40 SW_PUSH, SW41 SW_PUSH, SW42 SW_PUSH, SW43 SW_PUSH, SW44 SW_PUSH, SW45 SW_PUSH, SW46 SW_PUSH, SW47 SW_PUSH, SW48 SW_PUSH, SW49 SW_PUSH, SW5 SW_PUSH, SW50 SW_PUSH, SW51 SW_PUSH, SW52 SW_PUSH, SW53 SW_PUSH, SW54 SW_PUSH, SW55 SW_PUSH, SW6 SW_PUSH, SW7 SW_PUSH, SW8 SW_PUSH, SW9 SW_PUSH

Commit message: pcb
Parts:
- moved DS10 59.4 mm to (171.4, 51.6)
- moved D31 40.0 mm to (140.5, 29.8), turned to 180 degrees
- moved D43 35.5 mm to (140.5, 28.1), turned to 180 degrees
- moved D11 31.2 mm to (42.6, 73.5), turned to 180 degrees
- moved D10 30.7 mm to (43.0, 66.0), turned to 180 degrees
- moved D32 29.7 mm to (146.1, 55.0)
- moved D33 29.7 mm to (146.1, 56.8)
- moved DI6 28.4 mm to (43.7, 28.9)
- moved DS6 28.4 mm to (43.7, 27.4)
- moved D28 27.7 mm to (143.6, 51.4)
- moved D29 27.7 mm to (143.6, 53.2)
- moved D30 27.7 mm to (143.6, 55.0)
- moved D51 27.7 mm to (187.7, 77.5)
- moved DS5 25.8 mm to (59.9, 43.5), turned to 180 degrees
- moved DI5 21.0 mm to (43.7, 38.2)
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- renumbered REF**2 to Hole0, REF**7 to Hole1, REF**12 to Hole10, REF**3 to Hole11, REF**2 to Hole12, REF**5 to Hole2, REF**6 to Hole3, REF**4 to Hole4, REF**3 to Hole5, REF**8 to Hole6, REF**1 to Hole7, REF**13 to Hole8, REF**14 to Hole9
Routing:
- net GND_R: track 0.00 -> 178.7 mm, vias 0 -> 12
- net Pin11: track 0.00 -> 142.4 mm, vias 0 -> 3
- net Pin9: track 0.00 -> 125.9 mm, vias 0 -> 5
- net Pin3: track 0.00 -> 119.7 mm, vias 0 -> 4
- net Pin0: track 0.00 -> 119.0 mm, vias 0 -> 2
- net MOTION: track 0.00 -> 118.9 mm, vias 0 -> 5
- net Net-(D13-K): track 0.00 -> 117.8 mm, vias 0 -> 7
- net Pin8: track 0.00 -> 113.5 mm, vias 0 -> 6
- net Pin7: track 0.00 -> 111.6 mm, vias 0 -> 7
- net Pin5: track 0.00 -> 110.7 mm, vias 0 -> 3
- net Pin10: track 0.00 -> 108.3 mm, vias 0 -> 4
- net Net-(D11-K): track 0.00 -> 104.7 mm, vias 0 -> 6
- net SDIO: track 0.00 -> 98.2 mm, vias 0 -> 1
- net RE_B_L: track 0.00 -> 96.0 mm, vias 0 -> 5
- net 3.3V: track 0.00 -> 94.1 mm, vias 0 -> 10
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
Commit message: pcb
Parts:
- moved D30 41.8 mm to (111.2, 81.5), turned to 0 degrees
- moved D33 41.6 mm to (111.2, 79.4)
- moved D32 38.3 mm to (111.1, 70.5)
- moved D29 38.0 mm to (111.1, 73.0), turned to 0 degrees
- moved D1 37.5 mm to (35.7, 48.6), turned to 0 degrees
- moved D21 36.1 mm to (42.5, 73.0)
- moved D13 35.7 mm to (2.35, 34.0), turned to 0 degrees
- moved D5 33.5 mm to (2.35, 36.0)
- moved D9 29.7 mm to (2.35, 38.0)
- moved D40 24.4 mm to (152.8, 35.7), turned to 0 degrees
- moved DS1 20.1 mm to (52.8, 25.7), turned to 0 degrees
- moved D27 19.0 mm to (52.1, 72.2)
- moved D35 17.6 mm to (137.0, 27.9), turned to 180 degrees
- moved D26 14.6 mm to (42.5, 68.2)
- moved DS4 14.6 mm to (36.1, 68.2)
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Routing:
- net Net-(D13-K): track 117.8 -> 66.1 mm, vias 7 -> 4
- net Net-(D1-K): track 92.8 -> 45.3 mm, vias 5 -> 3
- net Net-(D29-K): track 85.3 -> 132.7 mm, vias 6 -> 10
- net Net-(D30-A): track 63.1 -> 18.5 mm
- net Net-(D33-A): track 50.7 -> 9.51 mm, vias 4 -> 0
- net Net-(D30-K): track 84.4 -> 119.6 mm, vias 5 -> 6
- net Net-(D13-A): track 47.1 -> 15.0 mm, vias 0 -> 2
- net Net-(D5-A): track 35.6 -> 6.23 mm
- net Net-(D27-A): track 60.5 -> 34.3 mm, vias 2 -> 0
- net Net-(D40-A): track 25.9 -> 3.25 mm, vias 2 -> 0
- net Net-(D11-K): track 104.7 -> 84.6 mm, vias 6 -> 4
- net Net-(D29-A): track 41.5 -> 21.7 mm
- net Net-(D23-A): track 11.7 -> 30.8 mm
- net Net-(D1-A): track 30.6 -> 48.0 mm, vias 0 -> 2
- net Net-(D35-A): track 33.3 -> 16.8 mm
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
Commit message: pcb
Connections:
- Con_L_0 pad 1: RE_B_L -> unconnected-(Con_L_0-Pin_1-Pad1)
- Con_L_0 pad 3: Pin5 -> Pin0
- Con_L_0 pad 4: Pin4 -> Pin1
- Con_L_10 pad 3: Pin9 -> Pin8
- Con_L_12 pad 4: Pin6 -> Pin11
- Con_L_14 pad 1: Pin7 -> Pin10
- Con_L_14 pad 2: Pin8 -> Pin9
- Con_L_2 pad 1: Pin3 -> unconnected-(Con_L_2-Pin_1-Pad1)
- Con_L_2 pad 2: RE_A_L -> unconnected-(Con_L_2-Pin_2-Pad2)
- Con_L_2 pad 4: Pin1 -> RE_A_L
- Con_L_4 pad 4: Pin0 -> Pin5
- Con_L_6 pad 1: unconnected-(Con_L_6-Pin_1-Pad1) -> Pin4
- Con_L_6 pad 2: unconnected-(Con_L_6-Pin_2-Pad2) -> Pin3
- Con_L_6 pad 3: unconnected-(Con_L_6-Pin_3-Pad3) -> RE_B_L
- Con_L_8 pad 3: Pin11 -> Pin6
- Con_L_8 pad 4: Pin10 -> Pin7
Routing:
- net RE_B_L: track 94.0 -> 39.6 mm, vias 3 -> 1
- net Pin9: track 123.4 -> 82.5 mm, vias 6 -> 4
- net Pin3: track 119.0 -> 154.1 mm, vias 4 -> 6
- net Pin7: track 112.3 -> 138.6 mm, vias 8 -> 10
- net Pin11: track 144.0 -> 119.8 mm, vias 5 -> 2
- net Pin4: track 86.0 -> 108.7 mm
- net Pin8: track 110.1 -> 131.7 mm, vias 6 -> 7
- net Pin0: track 129.3 -> 109.8 mm, vias 5 -> 6
- net Pin1: track 79.1 -> 95.6 mm, vias 5 -> 4
- net Net-(Con_L_9-Pin_2): track 32.6 -> 19.9 mm, vias 3 -> 2
- net Net-(D15-K): track 92.9 -> 81.7 mm, vias 7 -> 6
- net Net-(D29-K): track 132.7 -> 123.3 mm, vias 10 -> 9
- net Pin10: track 110.5 -> 101.4 mm, vias 6 -> 5
- net 3.3V: track 87.4 -> 82.0 mm, vias 8 -> 3
- net Pin2: track 84.1 -> 89.4 mm, vias 5 -> 3
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