File: PCB/nofy_Extensions/nofy.kicad_sch (KiCad schematic)
At the start: 144 parts, among them J10 Conn_01x01-Connector_Generic, J11 Conn_01x01-Connector_Generic, J12 Conn_01x01-Connector_Generic, J13 Conn_01x01-Connector_Generic, J14 Conn_01x01-Connector_Generic, J15 Conn_01x01-Connector_Generic, J16 Conn_01x01-Connector_Generic, J17 Conn_01x01-Connector_Generic, J18 Conn_01x01-Connector_Generic, J19 Conn_01x01-Connector_Generic, J20 Conn_01x01-Connector_Generic, J21 Conn_01x01-Connector_Generic, J22 PIn1x4, J23 PIn1x4, J24 PIn1x4, J25 PIn1x4, J26 PIn1x4, J27 PIn1x4, J28 PIn1x4, J29 PIn1x4, J30 PIn1x4, J31 PIn1x4, J32 PIn1x4, J33 PIn1x4, J34 PIn1x4, J35 PIn1x4, J36 PIn1x4, J37 PIn1x4, J38 PIn1x4, J39 PIn1x4, J40 PIn1x4, J41 PIn1x4, SW1 RotaryEncoder, SW10 SW_PUSH, SW11 SW_PUSH, SW12 SW_PUSH, SW13 SW_PUSH, SW14 SW_PUSH, SW15 SW_PUSH, SW16 SW_PUSH, SW17 SW_PUSH, SW18 SW_PUSH, SW19 SW_PUSH, SW2 RotaryEncoder, SW20 SW_PUSH, SW21 SW_PUSH, SW22 SW_PUSH, SW23 SW_PUSH, SW24 SW_PUSH, SW25 SW_PUSH, SW26 SW_PUSH, SW27 SW_PUSH, SW28 SW_PUSH, SW29 SW_PUSH, SW3 SW_SPDT, SW30 SW_PUSH, SW31 SW_PUSH, SW32 SW_PUSH, SW33 SW_PUSH, SW34 SW_PUSH, SW35 SW_PUSH, SW36 SW_PUSH, SW37 SW_PUSH, SW38 SW_PUSH, SW39 SW_PUSH, SW4 SW_SPDT, SW40 SW_PUSH, SW41 SW_PUSH, SW42 SW_PUSH, SW43 SW_PUSH, SW44 SW_PUSH, SW45 SW_PUSH, SW46 SW_PUSH, SW47 SW_PUSH, SW48 SW_PUSH, SW49 SW_PUSH, SW5 SW_PUSH, SW50 SW_PUSH, SW51 SW_PUSH, SW52 SW_PUSH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

Commit message: Update : PCB
Parts:
- J10, J11, J12, J13, J14, J15, J16, J17, J18, J19, J20, J21: footprint MountingHole:MountingHole_3.2mm_M3 -> nofy:MountingHole_2.2mm_M2
Changed lines of the file:
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@@
 			)
 		)
-		(property "Footprint" "MountingHole:MountingHole_3.2mm_M3"
+		(property "Footprint" "nofy:MountingHole_2.2mm_M2"
 			(at 217.17 228.6 0)
 			(effects
@@
 			)
 		)
-		(property "Footprint" "MountingHole:MountingHole_3.2mm_M3"
+		(property "Footprint" "nofy:MountingHole_2.2mm_M2"
 			(at 198.12 228.6 0)
 			(effects
@@
 			)
 		)
-		(property "Footprint" "MountingHole:MountingHole_3.2mm_M3"
+		(property "Footprint" "nofy:MountingHole_2.2mm_M2"
 			(at 285.75 113.03 0)
 			(effects
@@
 			)
 		)
-		(property "Footprint" "MountingHole:MountingHole_3.2mm_M3"
+		(property "Footprint" "nofy:MountingHole_2.2mm_M2"
 			(at 250.19 113.03 0)
 			(effects
@@
 			)
 		)
-		(property "Footprint" "MountingHole:MountingHole_3.2mm_M3"
+		(property "Footprint" "nofy:MountingHole_2.2mm_M2"
 			(at 213.36 113.03 0)
 			(effects
@@
 			)
 		)
-		(property "Footprint" "MountingHole:MountingHole_3.2mm_M3"
+		(property "Footprint" "nofy:MountingHole_2.2mm_M2"
 			(at 194.31 113.03 0)
 			(effects
@@
 			)
 		)
-		(property "Footprint" "MountingHole:MountingHole_3.2mm_M3"
+		(property "Footprint" "nofy:MountingHole_2.2mm_M2"
 			(at 254 228.6 0)
 			(effects
@@
 			)
 		)
-		(property "Footprint" "MountingHole:MountingHole_3.2mm_M3"
+		(property "Footprint" "nofy:MountingHole_2.2mm_M2"
 			(at 271.78 228.6 0)
 			(effects
@@
 			)
 		)
-		(property "Footprint" "MountingHole:MountingHole_3.2mm_M3"
+		(property "Footprint" "nofy:MountingHole_2.2mm_M2"
 			(at 267.97 113.03 0)
 			(effects
@@
 			)
 		)
-		(property "Footprint" "MountingHole:MountingHole_3.2mm_M3"
+		(property "Footprint" "nofy:MountingHole_2.2mm_M2"
 			(at 236.22 228.6 0)
 			(effects
@@
 			)
 		)
-		(property "Footprint" "MountingHole:MountingHole_3.2mm_M3"
+		(property "Footprint" "nofy:MountingHole_2.2mm_M2"
 			(at 232.41 113.03 0)
 			(effects
@@
 			)
 		)
-		(property "Footprint" "MountingHole:MountingHole_3.2mm_M3"
+		(property "Footprint" "nofy:MountingHole_2.2mm_M2"
 			(at 289.56 228.6 0)
 			(effects
