File: PCB/nofy_V2_R/nofy_V2_R.kicad_pcb (KiCad board)
At the start: 2 copper layers, 99.7 x 78.9 mm, 62 parts, among them J32 PIn1x4, SW32 SW_PUSH, SW33 SW_PUSH, SW34 SW_PUSH, SW35 SW_PUSH, SW36 SW_PUSH, SW37 SW_PUSH, SW39 SW_PUSH, SW4 RotaryEncoder, SW40 SW_PUSH, SW41 SW_PUSH, SW43 SW_PUSH, SW44 SW_PUSH, SW45 SW_PUSH, SW47 SW_PUSH, SW48 SW_PUSH, SW49 SW_PUSH, SW50 SW_PUSH, SW51 SW_PUSH, SW52 SW_PUSH, SW53 SW_PUSH, SW54 SW_PUSH, SW55 SW_PUSH

Commit message: pcb
Parts:
- added BT0: BATT_L, _kicad_footprints:JST_S2B-PH-SM4-TB, F.Cu at (223.6, 41.8)
- added BT1: BATT, _kicad_footprints:JST_S2B-PH-SM4-TB, F.Cu at (223.5, 74.2)
- added Con_L_0: PIn1x4, nofy:Pin1x4, F.Cu at (40.6, 16.3)
- added Con_L_1: PIn1x4, nofy:Pin1x4, F.Cu at (214.8, 24.6)
- added Con_L_11: PIn1x4, nofy:Pin1x4, F.Cu at (251.4, 68.6)
- added Con_L_13: PIn1x4, nofy:Pin1x4, F.Cu at (217.4, 93.4)
- added Con_L_15: PIn1x4, nofy:Pin1x4, F.Cu at (217.4, 76.4)
- added Con_L_2: PIn1x4, nofy:Pin1x4, F.Cu at (40.6, 31.4)
- added Con_L_3: PIn1x4, nofy:Pin1x4, F.Cu at (214.8, 39.8)
- added Con_L_4: PIn1x4, nofy:Pin1x4, F.Cu at (74.6, 24.4)
- added Con_L_5: PIn1x4, nofy:Pin1x4, F.Cu at (248.8, 32.8)
- added Con_L_6: PIn1x4, nofy:Pin1x4, F.Cu at (74.6, 39.5)
- added Con_L_7: PIn1x4, nofy:Pin1x4, F.Cu at (248.8, 47.8)
- added Con_L_9: PIn1x4, nofy:Pin1x4, F.Cu at (251.4, 85.3)
- added D1: D, _kicad_footprints:Diode_SMD, F.Cu at (35.7, 48.6)
- added D10: D, _kicad_footprints:Diode_SMD, F.Cu at (36.2, 58.5)
- added D11: D, _kicad_footprints:Diode_SMD, F.Cu at (42.5, 70.7)
- added D12: D, _kicad_footprints:Diode_SMD, F.Cu at (266.2, 60.9)
- added D13: D, _kicad_footprints:Diode_SMD, F.Cu at (2.35, 34.0)
- added D14: D, _kicad_footprints:Diode_SMD, F.Cu at (49.8, 32.9)
- added D15: D, _kicad_footprints:Diode_SMD, F.Cu at (57.0, 40.4)
- added D16: D, _kicad_footprints:Diode_SMD, F.Cu at (52.1, 70.1)
- added D17: D, _kicad_footprints:Diode_SMD, F.Cu at (53.1, 77.9)
- added D18: D, _kicad_footprints:Diode_SMD, F.Cu at (56.2, 27.2)
- added D19: D, _kicad_footprints:Diode_SMD, F.Cu at (49.8, 35.0)
- added D2: D, _kicad_footprints:Diode_SMD, F.Cu at (10.8, 65.3)
- added D20: D, _kicad_footprints:Diode_SMD, F.Cu at (56.9, 38.5)
- added D21: D, _kicad_footprints:Diode_SMD, F.Cu at (42.5, 73.0)
- added D22: D, _kicad_footprints:Diode_SMD, F.Cu at (53.1, 75.8)
- added D23: D, _kicad_footprints:Diode_SMD, F.Cu at (56.2, 24.1)
- added D24: D, _kicad_footprints:Diode_SMD, F.Cu at (43.6, 50.3)
- added D25: D, _kicad_footprints:Diode_SMD, F.Cu at (43.6, 52.0)
- added D26: D, _kicad_footprints:Diode_SMD, F.Cu at (42.5, 68.2)
- added D27: D, _kicad_footprints:Diode_SMD, F.Cu at (52.1, 72.2)
- added D3: D, _kicad_footprints:Diode_SMD, F.Cu at (3.35, 70.8)
- added D34: D, _kicad_footprints:Diode_SMD, F.Cu at (292.5, 46.9)
- added D38: D, _kicad_footprints:Diode_SMD, F.Cu at (275.5, 46.9)
- added D4: D, _kicad_footprints:Diode_SMD, F.Cu at (300.4, 61.0)
- added D42: D, _kicad_footprints:Diode_SMD, F.Cu at (258.5, 46.8)
- added D5: D, _kicad_footprints:Diode_SMD, F.Cu at (2.35, 36.0)
- added D6: D, _kicad_footprints:Diode_SMD, F.Cu at (10.8, 63.0)
- added D7: D, _kicad_footprints:Diode_SMD, F.Cu at (3.35, 68.4)
- added D8: D, _kicad_footprints:Diode_SMD, F.Cu at (283.3, 61.0)
- added D9: D, _kicad_footprints:Diode_SMD, F.Cu at (2.35, 38.0)
- added DI1: D, _kicad_footprints:Diode_SMD, F.Cu at (43.7, 30.9)
- added DI2: D, _kicad_footprints:Diode_SMD, F.Cu at (43.7, 32.9)
- added DI3: D, _kicad_footprints:Diode_SMD, F.Cu at (43.7, 34.9)
- added DI4: D, _kicad_footprints:Diode_SMD, F.Cu at (43.7, 36.8)
- added DI5: D, _kicad_footprints:Diode_SMD, F.Cu at (43.7, 38.7)
- added DI6: D, _kicad_footprints:Diode_SMD, F.Cu at (43.7, 28.9)
- added DS1: D, _kicad_footprints:Diode_SMD, F.Cu at (52.8, 25.7)
- added DS2: D, _kicad_footprints:Diode_SMD, F.Cu at (35.8, 50.4)
- added DS3: D, _kicad_footprints:Diode_SMD, F.Cu at (35.8, 52.0)
- added DS4: D, _kicad_footprints:Diode_SMD, F.Cu at (36.1, 68.2)
- added DS5: D, _kicad_footprints:Diode_SMD, F.Cu at (57.1, 42.5)
- added DS6: D, _kicad_footprints:Diode_SMD, F.Cu at (43.7, 27.4)
- added Hole0: MountingHole_2.2mm_M2, nofy:MountingHole_2.2mm_M2, F.Cu at (7.40, 41.2)
- added Hole1: MountingHole_2.2mm_M2, nofy:MountingHole_2.2mm_M2, F.Cu at (7.50, 75.2)
- added Hole10: MountingHole_2.2mm_M2, nofy:MountingHole_2.2mm_M2, F.Cu at (268.4, 51.4)
- added Hole11: MountingHole_2.2mm_M2, nofy:MountingHole_2.2mm_M2, F.Cu at (290.2, 47.6)
- added Hole12: MountingHole_2.2mm_M2, nofy:MountingHole_2.2mm_M2, F.Cu at (239.2, 54.1)
- added Hole2: MountingHole_2.2mm_M2, nofy:MountingHole_2.2mm_M2, F.Cu at (59.1, 52.9)
- added Hole3: MountingHole_2.2mm_M2, nofy:MountingHole_2.2mm_M2, F.Cu at (59.2, 69.3)
- added Hole7: MountingHole_2.2mm_M2, nofy:MountingHole_2.2mm_M2, F.Cu at (224.1, 33.2)
- added Hole8: MountingHole_2.2mm_M2, nofy:MountingHole_2.2mm_M2, F.Cu at (233.5, 65.7)
- added Hole9: MountingHole_2.2mm_M2, nofy:MountingHole_2.2mm_M2, F.Cu at (225.8, 92.7)
- added J18: PIn1x4, nofy:Pin1x4, F.Cu at (6.62, 50.9)
- added J21: PIn1x4, nofy:Pin1x4, F.Cu at (287.4, 49.8)
- added J33: PIn1x4, nofy:Pin1x4, F.Cu at (281.6, 46.6)
- added SW1: SW_SPDT, _kicad_footprints:TGSW_MSK-12D19, F.Cu at (224.3, 24.4)
- added SW10: SW_PUSH, nofy:Choc_v2_Hotswap_1u_17mm, F.Cu at (16.4, 58.5)
- added SW11: SW_PUSH, nofy:Choc_v2_Hotswap_1u_17mm, F.Cu at (16.4, 75.5)
- added SW12: SW_PUSH, nofy:Choc_v2_Hotswap_1u_17mm, F.Cu at (277.1, 59.4)
- added SW13: SW_PUSH, nofy:Choc_v2_Hotswap_1u_17mm, F.Cu at (33.4, 38.4)
- added SW14: SW_PUSH, nofy:Choc_v2_Hotswap_1u_17mm, F.Cu at (33.4, 55.4)
- added SW15: SW_PUSH, nofy:Choc_v2_Hotswap_1u_17mm, F.Cu at (33.4, 72.4)
- added SW16: SW_PUSH, nofy:Choc_v2_Hotswap_1u_17mm, F.Cu at (260.1, 59.4)
- added SW17: SW_PUSH, nofy:Choc_v2_Hotswap_1u_17mm, F.Cu at (-0.60, 32.7)
- added SW18: SW_PUSH, nofy:Choc_v2_Hotswap_1u_17mm, F.Cu at (50.4, 24.5)
- added SW19: SW_PUSH, nofy:Choc_v2_Hotswap_1u_17mm, F.Cu at (50.4, 41.5)
- added SW2: SW_SPDT, _kicad_footprints:TGSW_MSK-12D19, F.Cu at (224.5, 101.9)
- added SW20: SW_PUSH, nofy:Choc_v2_Hotswap_1u_17mm, F.Cu at (50.4, 58.5)
- added SW21: SW_PUSH, nofy:Choc_v2_Hotswap_1u_17mm, F.Cu at (50.4, 75.5)
- added SW22: SW_PUSH, nofy:Choc_v2_Hotswap_1u_17mm, F.Cu at (16.4, 24.5)
- added SW23: SW_PUSH, nofy:Choc_v2_Hotswap_1u_17mm, F.Cu at (67.4, 26.9)
- added SW24: SW_PUSH, nofy:Choc_v2_Hotswap_1u_17mm, F.Cu at (67.4, 43.9)
- added SW25: SW_PUSH, nofy:Choc_v2_Hotswap_1u_17mm, F.Cu at (67.4, 60.9)
- added SW26: SW_PUSH, nofy:Choc_v2_Hotswap_1u_17mm, F.Cu at (67.4, 77.9)
- added SW27: SW_PUSH, nofy:Choc_v2_Hotswap_1u_17mm, F.Cu at (33.4, 21.4)
- added SW28: SW_PUSH, nofy:Choc_v2_Hotswap_1u_17mm, F.Cu at (84.4, 32.7)
- added SW29: SW_PUSH, nofy:Choc_v2_Hotswap_1u_17mm, F.Cu at (84.4, 49.7)
- added SW3: RotaryEncoder, nofy:RotaryEncoder_EC12E, B.Cu at (68.3, 79.7)
- added SW30: SW_PUSH, nofy:Choc_v2_Hotswap_1u_17mm, F.Cu at (84.4, 66.7)
- added SW31: SW_PUSH, nofy:Choc_v2_Hotswap_1u_17mm, F.Cu at (84.4, 83.7)
- added SW38: SW_PUSH, nofy:Choc_v2_Hotswap_1u_17mm, F.Cu at (298.8, 39.6)
- added SW42: SW_PUSH, nofy:Choc_v2_Hotswap_1u_17mm, F.Cu at (281.8, 39.6)
- added SW46: SW_PUSH, nofy:Choc_v2_Hotswap_1u_17mm, F.Cu at (264.8, 39.6)
- added SW5: SW_PUSH, nofy:Choc_v2_Hotswap_1u_17mm, F.Cu at (-0.60, 49.7)
- added SW6: SW_PUSH, nofy:Choc_v2_Hotswap_1u_17mm, F.Cu at (-0.60, 66.7)
- added SW7: SW_PUSH, nofy:Choc_v2_Hotswap_1u_17mm, F.Cu at (-0.60, 83.7)
- added SW8: SW_PUSH, nofy:Choc_v2_Hotswap_1u_17mm, F.Cu at (294.1, 59.4)
- added SW9: SW_PUSH, nofy:Choc_v2_Hotswap_1u_17mm, F.Cu at (16.4, 41.5)
- added Xiao0: ~, _kicad_footprints:XIAO_nRF52840_wBAT_wNFC_1, F.Cu at (239.3, 26.8)
- added Xiao1: ~, _kicad_footprints:XIAO_nRF52840_wBAT_wNFC_1, F.Cu at (239.3, 99.5)
- D28, D29, D30, D31, D32, D33, D35, D36, D37, D39, D40, D41, D43, D44, D45, D46, D47, D48, D49, D50, D51, DI10, DI11, DI7, DI8, DI9, DS10, DS11, DS7, DS8, DS9: moved to F.Cu
- moved D44 90.3 mm to (185.7, 28.8)
- moved D41 88.3 mm to (184.6, 47.2), turned to 0 degrees
- moved D45 88.1 mm to (184.6, 45.4)
- moved D48 85.4 mm to (185.7, 30.9)
- moved D49 81.7 mm to (184.6, 49.2)
- moved DS8 81.6 mm to (149.3, 37.5)
- moved DI7 81.2 mm to (140.8, 27.9)
- moved DI8 81.2 mm to (140.8, 29.9)
- moved DI9 81.2 mm to (140.8, 31.8)
- moved DI10 81.1 mm to (140.8, 33.8)
- moved D28 81.1 mm to (143.7, 51.6), turned to 0 degrees
- moved DI11 81.1 mm to (140.8, 35.7)
- moved DS11 81.1 mm to (140.8, 37.7)
- moved Con_L_12 81.0 mm to (150.8, 24.5)
- moved Con_L_14 81.0 mm to (150.8, 41.6)
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Routing:
- net Pin0: track 0.00 -> 129.3 mm, vias 0 -> 5
- net Pin3: track 0.00 -> 119.0 mm, vias 0 -> 4
- net Pin5: track 0.00 -> 110.7 mm, vias 0 -> 8
- net Net-(D16-K): track 0.00 -> 102.1 mm, vias 0 -> 8
- net RE_B_L: track 0.00 -> 94.0 mm, vias 0 -> 3
- net Net-(D15-K): track 0.00 -> 92.9 mm, vias 0 -> 7
- net Pin4: track 0.00 -> 86.0 mm, vias 0 -> 3
- net Net-(D11-K): track 0.00 -> 84.6 mm, vias 0 -> 4
- net Pin2: track 0.00 -> 84.1 mm, vias 0 -> 5
- net Pin1: track 0.00 -> 79.1 mm, vias 0 -> 5
- net RE_A_L: track 0.00 -> 75.4 mm, vias 0 -> 3
- net Net-(D13-K): track 0.00 -> 66.1 mm, vias 0 -> 4
- net Net-(D18-A): track 0.00 -> 60.1 mm, vias 0 -> 2
- net Net-(D17-K): track 0.00 -> 57.8 mm
- net GND_L: track 0.00 -> 52.9 mm
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Other:
- board size 99.7 x 78.9 mm -> 314.7 x 88.7 mm
- board text added: "L"
- board text added: "R"
- board text added: "nofy Engine"

Commit message: pcb
Parts:
- removed BT0: BATT_L, _kicad_footprints:JST_S2B-PH-SM4-TB
- removed BT1: BATT, _kicad_footprints:JST_S2B-PH-SM4-TB
- removed Con_L_0, Con_L_1, Con_L_11, Con_L_13, Con_L_15, Con_L_2, Con_L_3, Con_L_4, Con_L_5, Con_L_6, Con_L_7, Con_L_9, J18, J21, J33: PIn1x4, nofy:Pin1x4
- removed D1, D10, D11, D12, D13, D14, D15, D16, D17, D18, D19, D2, D20, D21, D22, D23, D24, D25, D26, D27, D3, D34, D38, D4, D42, D5, D6, D7, D8, D9, DI1, DI2, DI3, DI4, DI5, DI6, DS1, DS2, DS3, DS4, DS5, DS6: D, _kicad_footprints:Diode_SMD
- removed Hole0, Hole1, Hole10, Hole11, Hole12, Hole2, Hole3, Hole7, Hole8, Hole9: MountingHole_2.2mm_M2, nofy:MountingHole_2.2mm_M2
- removed SW1, SW2: SW_SPDT, _kicad_footprints:TGSW_MSK-12D19
- removed SW10, SW11, SW12, SW13, SW14, SW15, SW16, SW17, SW18, SW19, SW20, SW21, SW22, SW23, SW24, SW25, SW26, SW27, SW28, SW29, SW30, SW31, SW38, SW42, SW46, SW5, SW6, SW7, SW8, SW9: SW_PUSH, nofy:Choc_v2_Hotswap_1u_17mm
- removed SW3: RotaryEncoder, nofy:RotaryEncoder_EC12E
- removed Xiao0, Xiao1: ~, _kicad_footprints:XIAO_nRF52840_wBAT_wNFC_1
Connections:
- Con_L_10 pad 3: Pin9 -> Pin8
- Con_L_12 pad 4: Pin6 -> Pin11
- Con_L_14 pad 1: Pin7 -> Pin10
- Con_L_14 pad 2: Pin8 -> Pin9
- Con_L_8 pad 3: Pin11 -> Pin6
- Con_L_8 pad 4: Pin10 -> Pin7
Routing:
- net Pin0: track 129.3 -> 0.00 mm, vias 5 -> 0
- net Pin3: track 119.0 -> 0.00 mm, vias 4 -> 0
- net Pin5: track 110.7 -> 0.00 mm, vias 8 -> 0
- net Net-(D16-K): track 102.1 -> 0.00 mm, vias 8 -> 0
- net RE_B_L: track 94.0 -> 0.00 mm, vias 3 -> 0
- net Net-(D15-K): track 92.9 -> 0.00 mm, vias 7 -> 0
- net Pin4: track 86.0 -> 0.00 mm, vias 3 -> 0
- net Net-(D11-K): track 84.6 -> 0.00 mm, vias 4 -> 0
- net Pin2: track 84.1 -> 0.00 mm, vias 5 -> 0
- net Pin1: track 79.1 -> 0.00 mm, vias 5 -> 0
- net RE_A_L: track 75.4 -> 0.00 mm, vias 3 -> 0
- net Net-(D13-K): track 66.1 -> 0.00 mm, vias 4 -> 0
- net Net-(D18-A): track 60.1 -> 0.00 mm, vias 2 -> 0
- net Net-(D17-K): track 57.8 -> 0.00 mm
- net GND_L: track 52.9 -> 0.00 mm
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Other:
- board size 314.7 x 88.7 mm -> 99.7 x 78.9 mm
- board text removed: "L"
- board text removed: "R"
- board text removed: "nofy Engine"
